File: SnarkBarker.sch (KiCad schematic (older format))
At the start: 194 parts, among them J1 Bus_ISA_8bit, J2 Bracket Mount, P1 Joystick/MIDI, P2 L7809, T1 2N3904, T2 2N3904, U1 NE558, U10 YM3014B, U11 NJM3403A, U12 MC1408_DIP, U13 805X, U14 SAA1099, U15 SAA1099, U16 74LS08, U17 74LS139, U18 74LS374, U19 74LS374, U2 74LS245, U20 74LS74, U21 74LS125, U22 74LS74, U23 74LS74, U24 74LS32, U25 74LS08, U26 74LS74, U27 74LS32, U28 74LS08, U29 74LS14, U3 74LS244, U30 74LS32, U4 TEA2025B, U5 LM324, U6 LM393, U7 74LS138, U8 74LS138, U9 YM3812

Commit message: Swap out obsolete parts P1 and U5
Parts:
- P1: Mouser 152-3415 -> 1636-182-015-213R53
- U5: Mouser 512-LM324AN -> 595-LM324AN
Changed lines of the file:
@@
 F 2 "SoundBlaster:SB_DIP14_300" H 7600 11850 50  0001 C CNN
 F 3 "" H 7700 11950 50  0001 C CNN
-F 4 "512-LM324AN" H 7650 11750 60  0001 C CNN "Mouser"
+F 4 "595-LM324AN" H 7650 11750 60  0001 C CNN "Mouser"
 	1    7650 11750
 	1    0    0    1
@@
 F 2 "SoundBlaster:SB_DB15_152-3415" H 15700 7000 50  0001 C CNN
 F 3 "" H 15700 7000 50  0001 C CNN
-F 4 "152-3415" H 15700 7000 60  0001 C CNN "Mouser"
+F 4 "1636-182-015-213R53" H 15700 7000 60  0001 C CNN "Mouser"
 	1    15700 7000
 	1    0    0    -1
